Commit message: update gpu vlp

File: scout_description/urdf/accessories/vlp16_mount.urdf.xacro (robot description, xacro)
@@ -2,5 +2,5 @@
 <robot xmlns:xacro="http://wiki.ros.org/xacro">
   <xacro:include filename="$(find velodyne_description)/urdf/VLP-16.urdf.xacro" />
-  <xacro:macro name="vlp16_mount" params="prefix parent_link topic height:=0.12 *origin">
+  <xacro:macro name="vlp16_mount" params="prefix parent_link topic gpu height:=0.12 *origin">
     <!--
       The VLP16 is mounted to a pair of extrusion rods on top of the main sensor arch
@@ -78,5 +78,5 @@
       <origin xyz="0 0 ${height}" rpy="0 0 0"/>
     </joint>
-    <xacro:VLP-16 parent="${prefix}vlp16_mount_plate" topic="${topic}">
+    <xacro:VLP-16 parent="${prefix}vlp16_mount_plate" topic="${topic}" gpu="${gpu}">
       <origin xyz="0 0 0" rpy="0 0 0" />
     </xacro:VLP-16>

File: scout_description/urdf/scout_v2.xacro (robot description, xacro)
@@ -91,7 +91,7 @@
         <child link="base_laser_mount" />
         </joint>
-        <!-- <xacro:vlp16_mount prefix="" parent_link="base_link" topic="points">
-        <origin xyz="-0.2 0 0.4" rpy="0 0 0" />
-        </xacro:vlp16_mount> -->
+        <xacro:vlp16_mount prefix="base" parent_link="base_link" topic="velodyne_points" gpu="true">
+        <origin xyz="0.4 0 0.4" rpy="0 0 0" />
+        </xacro:vlp16_mount>
     </xacro:if>
 </robot>
